File: ZEUS WPT/zeuswpt/zeuswpt.kicad_sch (KiCad schematic)
At the start: 0 parts

Commit message: Update ZEUS WPT
Parts:
- added U1: VSC5-2805S, Converter_DCDC:Converter_DCDC_Silvertel_Ag99xxLP_THT, symbol Converter_DCDC:Ag9905LP
- added U2: WVA-44603LN+, Package_TO_SOT_SMD:SOT-363_SC-70-6, symbol RF_Amplifier:BGA2867
Connections:
- new net: U2.2 (G), U2.4 (G), U2.5 (G)
- new net: U1.5 (VIN+), U1.6 (VIN+), U2.3
- new net: U1.1 (+VDC), U1.2 (+VDC)
- new net: U1.7 (VIN-), U1.8 (VIN-)
- new net GND: U2.1 (Vcc)
Other:
- note added: "50VDC PCDU Power Bus"
- note added: "Cooling System"
- note added: "EPS"
- note added: "Feedback Loop"
- note added: "Phased Arrays (x12)"
- note added: "Thermoelectric Generator"
