File: ZEUS WPT/zeuswpt/zeuswpt.kicad_sch (KiCad schematic)
At the start: 2 parts, among them U1 VSC5-2805S, U2 WVA-44603LN+

Commit message: EPS v3 et WPT v2
Parts:
- removed U2: WVA-44603LN+, Package_TO_SOT_SMD:SOT-363_SC-70-6, symbol RF_Amplifier:BGA2867
Other:
- note added: "50VDC PCDU Unregulated"
- note added: "DC-DC Converter"
- note added: "Passive Cooling System"
- note added: "STELLAR High Power (x2)"
- note added: "Traveling-Wave Tube Amplifier"
- note removed: "50VDC PCDU Power Bus"
- note removed: "Cooling System"
- note removed: "EPS"
- note removed: "Thermoelectric Generator"
- moved on the sheet: U1

Commit message: Update
Parts:
- removed U1: VSC5-2805S, Converter_DCDC:Converter_DCDC_Silvertel_Ag99xxLP_THT, symbol Converter_DCDC:Ag9905LP
Other:
- note added: "11/8/2024"
- note added: "Axial to Coaxial Converter"
- note added: "Phased Arrays (x4)"
- note added: "Traveling-Wave Tube Amplifier (x5)"
- note added: "Waveguide Bandpass Filter"
- note removed: "4/8/2024"
- note removed: "DC-DC Converter"
- note removed: "Feedback Loop"
- note removed: "Phased Arrays (x12)"
- note removed: "Traveling-Wave Tube Amplifier"
