File: ZEUS EPS/EPS_v1.kicad_sch (KiCad schematic)
At the start: 6 parts, among them U1 XL1509-3.3

Commit message: EPS v3 et WPT v2
Parts:
- added BT2: StellarBatt, symbol Device:Battery
Connections:
- net GND: now also BT2.2 (-)
- net at BT1.1 (+), U1.1 (VIN): now also BT2.1 (+)
Other:
- note added: "28V Regulated"
- note added: "STELLAR Batt (x2) 22.7 - 37.8V 36.9 during Cycling operations"
- note added: "Secondary Battery Nom. 4.2V Standard. 3.63V Discharge : 2.5V"
- note removed: "28V Unregulated"
- note removed: "Stellar Batt 22.7 - 37.8V 36.9 during Cycling operations"
- moved on the sheet: BT1
